Commit message: Version 1.0.3

File: pi_hexapod_driver-1.0.2/pi_hexapod_description/urdf/pi_hexapod.macro.xacro (robot description, xacro)
@@ -109,5 +109,4 @@
                        ${hexapod_parameters['platform']['visual']['scale']}" />
         </geometry>
-        <material name="gray" />
       </visual>
        <collision>
